File: kiCad/schema/schema.kicad_sch (KiCad schematic)
At the start: 0 parts

Commit message: Day 4
Parts:
- added J1: Esp32, symbol Connector_Generic:Conn_02x15_Counter_Clockwise
- added J10: IR 4, symbol Connector_Generic:Conn_01x03
- added J11: Switch, symbol Connector:Conn_01x02_Pin
- added J2: DRV8833, symbol Connector_Generic:Conn_02x06_Counter_Clockwise
- added J3: M1 Right, symbol Connector:Conn_01x06_Pin
- added J4: M2 Left, symbol Connector:Conn_01x06_Pin
- added J5: Bat, symbol Connector_Generic:Conn_01x02
- added J6: Buck, symbol Connector_Generic:Conn_01x04
- added J7: IR 1, symbol Connector_Generic:Conn_01x03
- added J8: IR 3, symbol Connector_Generic:Conn_01x03
- added J9: IR 2, symbol Connector_Generic:Conn_01x03
Connections:
- new net AIN 1: J1.9 (Pin_9), J2.7 (Pin_7)
- new net AIN 2: J1.10 (Pin_10), J2.8 (Pin_8)
- new net AOUT 1: J2.2 (Pin_2)
- new net AOUT 2: J2.3 (Pin_3)
- new net BAT +: J11.1 (Pin_1), J5.1 (Pin_1), J6.1 (Pin_1)
- new net BAT -: J5.2 (Pin_2), J6.2 (Pin_2)
- new net BIN 1: J1.11 (Pin_11), J2.11 (Pin_11)
- new net BIN 2: J1.12 (Pin_12), J2.12 (Pin_12)
- new net BOUT 1: J2.4 (Pin_4)
- new net BOUT 2: J2.5 (Pin_5)
- new net BUCK +: J1.15 (Pin_15), J6.3 (Pin_3)
- new net BUCk -: J6.4 (Pin_4)
- new net GND: J1.30 (Pin_30), J10.2 (Pin_2), J2.10 (Pin_10), J3.5 (Pin_5), J4.5 (Pin_5), J7.2 (Pin_2), J8.2 (Pin_2), J9.2 (Pin_2)
- new net IR 1: J7.3 (Pin_3)
- new net IR 3: J8.3 (Pin_3), J9.3 (Pin_3)
- new net IR 4: J10.3 (Pin_3)
- new net OUT: J10.1 (Pin_1), J11.2 (Pin_2), J2.9 (Pin_9), J7.1 (Pin_1), J8.1 (Pin_1), J9.1 (Pin_1)

Commit message: Day 6 - Schematics
Connections:
- net BUCk - is gone; now on net GND: J6.4 (Pin_4)
- net AIN 1: now also J1.8 (Pin_8); no longer J1.9 (Pin_9)
- net AIN 2: now also J1.9 (Pin_9); no longer J1.10 (Pin_10)
- net AOUT 1: now also J3.1 (Pin_1)
- net AOUT 2: now also J3.6 (Pin_6)
- net BAT +: no longer J11.1 (Pin_1), J5.1 (Pin_1)
- net BAT -: no longer J5.2 (Pin_2)
- net BIN 1: now also J1.10 (Pin_10); no longer J1.11 (Pin_11)
- net BIN 2: now also J1.11 (Pin_11); no longer J1.12 (Pin_12)
- net BOUT 1: now also J4.1 (Pin_1)
- net BOUT 2: now also J4.6 (Pin_6)
- net BUCK +: now also J10.1 (Pin_1), J3.2 (Pin_2), J4.2 (Pin_2), J7.1 (Pin_1), J8.1 (Pin_1), J9.1 (Pin_1)
- net GND: now also J1.14 (Pin_14), J1.17 (Pin_17), J5.2 (Pin_2); no longer J1.30 (Pin_30)
- net IR 1: now also J1.2 (Pin_2)
- net IR 3: now also J1.20 (Pin_20); no longer J9.3 (Pin_3)
- net IR 4: now also J1.23 (Pin_23)
- net OUT: no longer J10.1 (Pin_1), J7.1 (Pin_1), J8.1 (Pin_1), J9.1 (Pin_1)
- net IR 2: now reaches J1.3 (Pin_3)
- net IR 2: now also J9.3 (Pin_3)
- net ENC A1: now reaches J1.4 (Pin_4)
- net ENC A1: now also J3.3 (Pin_3)
- net ENC A2: now reaches J1.5 (Pin_5)
- net ENC A2: now also J3.4 (Pin_4)
- net ENC B1: now reaches J1.6 (Pin_6)
- net ENC B1: now also J4.3 (Pin_3)
- net ENC B2: now reaches J1.7 (Pin_7)
- net ENC B2: now also J4.4 (Pin_4)
- new net VCC: J11.1 (Pin_1), J5.1 (Pin_1)
- no-connect marks 0 -> 15
Other:
- moved on the sheet: J3, J4, J5

Commit message: Day 7 - Schematics finished
Parts:
- added C1, C3: C, symbol Device:C
- added C2: C_Polarized, symbol Device:C_Polarized
Connections:
- net BAT - is gone; now on net GND: J6.2 (Pin_2)
- net OUT is gone; now on net BAT +: J11.2 (Pin_2), J2.9 (Pin_9)
- net BAT +: now also C3.2
- net BUCK +: now also J2.1 (Pin_1), C1.2, C2.1
- net GND: now also C1.1, C2.2, C3.1
- net VCC renamed BAT R+
- no-connect marks 15 -> 16
Other:
- note added: "ESP32"
- note added: "IR SENSORS"
- note added: "MOTOR AND DRIVER"
- note added: "POWER SUPPLY"
- moved on the sheet: J1, J10, J11, J2, J3, J4, J5, J6, J7, J8, J9

Commit message: Day 8 - Research, CAD design
Parts:
- J1: footprint (none) -> Connector_PinHeader_2.54mm:PinHeader_1x15_P2.54mm_Vertical
Other:
- moved on the sheet: J4

Commit message: Day 10 - CAD design, PCB design started
Parts:
- removed J1: Esp32, Connector_PinHeader_2.54mm:PinHeader_1x15_P2.54mm_Vertical, symbol Connector_Generic:Conn_02x15_Counter_Clockwise
- added J12, J13: Conn_01x15_Pin, Connector_PinHeader_2.54mm:PinHeader_1x15_P2.54mm_Vertical, symbol Connector:Conn_01x15_Pin
Connections:
- net AIN 1: now also J12.8 (Pin_8)
- net AIN 2: now also J12.9 (Pin_9)
- net BIN 1: now also J12.10 (Pin_10)
- net BIN 2: now also J12.11 (Pin_11)
- net BUCK +: now also J12.15 (Pin_15)
- net ENC A1: now also J12.4 (Pin_4)
- net ENC A2: now also J12.5 (Pin_5)
- net ENC B1: now also J12.6 (Pin_6)
- net ENC B2: now also J12.7 (Pin_7)
- net GND: now also J12.14 (Pin_14), J13.2 (Pin_2)
- net IR 1: now also J12.2 (Pin_2)
- net IR 2: now also J12.3 (Pin_3)
- net IR 3: now also J13.5 (Pin_5)
- net IR 4: now also J13.8 (Pin_8)
Other:
- moved on the sheet: C1, C2

Commit message: Day 11 -- PCB, footprints, headache
Parts:
- C1, C3: footprint (none) -> Capacitor_THT:C_Disc_D3.0mm_W1.6mm_P2.50mm
- C2: footprint (none) -> Capacitor_THT:CP_Radial_D4.0mm_P1.50mm
- J3, J4: footprint (none) -> Connector_PinHeader_2.54mm:PinHeader_1x06_P2.54mm_Vertical
Changed lines of the file:
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@@
 			)
 		)
-		(property "Footprint" ""
+		(property "Footprint" "Capacitor_THT:C_Disc_D3.0mm_W1.6mm_P2.50mm"
 			(at 183.8452 77.47 0)
 			(hide yes)
@@
 			)
 		)
-		(property "Footprint" ""
+		(property "Footprint" "Connector_PinHeader_2.54mm:PinHeader_1x06_P2.54mm_Vertical"
 			(at 180.34 95.25 0)
 			(hide yes)
@@
 			)
 		)
-		(property "Footprint" ""
+		(property "Footprint" "Capacitor_THT:CP_Radial_D4.0mm_P1.50mm"
 			(at 85.3948 97.79 0)
 			(hide yes)
@@
 			)
 		)
-		(property "Footprint" ""
+		(property "Footprint" "Connector_PinHeader_2.54mm:PinHeader_1x06_P2.54mm_Vertical"
 			(at 148.59 95.25 0)
 			(hide yes)
@@
 			)
 		)
-		(property "Footprint" ""
+		(property "Footprint" "Capacitor_THT:C_Disc_D3.0mm_W1.6mm_P2.50mm"
 			(at 93.6752 105.41 0)
 			(hide yes)

Commit message: Day 12 -- Resuming the project
Parts:
- removed J2: DRV8833, symbol Connector_Generic:Conn_02x06_Counter_Clockwise
- added J1, J14: Conn_01x06_Pin, Connector_PinHeader_2.54mm:PinHeader_1x06_P2.54mm_Vertical, symbol Connector:Conn_01x06_Pin
- added R1: 100 ohm, symbol Device:R
- J11: footprint (none) -> Button_Switch_THT:SW_Slide_SPDT_Straight_CK_OS102011MS2Q
- J5: footprint (none) -> Connector_JST:JST_PH_B2B-PH-K_1x02_P2.00mm_Vertical
- J6: footprint (none) -> Connector_PinHeader_2.54mm:PinHeader_1x02_P2.54mm_Vertical
Connections:
- net AIN 1: now also J14.1 (Pin_1)
- net AIN 2: now also J14.2 (Pin_2)
- net AOUT 1: now also J1.2 (Pin_2)
- net AOUT 2: now also J1.3 (Pin_3)
- net BAT +: now also J14.3 (Pin_3)
- net BIN 1: now also J14.5 (Pin_5)
- net BIN 2: now also J14.6 (Pin_6)
- net BOUT 1: now also J1.4 (Pin_4)
- net BOUT 2: now also J1.5 (Pin_5)
- net BUCK +: now also J1.1 (Pin_1)
- net GND: now also J14.4 (Pin_4)
- new net IR EM: R1.1
Other:
- moved on the sheet: C3

Commit message: Day 13 -- IR leds, footprints
Parts:
- removed J10: IR 4, symbol Connector_Generic:Conn_01x03
- removed J7: IR 1, symbol Connector_Generic:Conn_01x03
- removed J8: IR 3, symbol Connector_Generic:Conn_01x03
- removed J9: IR 2, symbol Connector_Generic:Conn_01x03
- added D1, D2, D3, D4: LED, LED_THT:LED_D5.0mm_Clear, symbol Device:LED
- added J15: MOSFET, symbol Connector_Generic:Conn_01x03
- added Q1, Q2, Q3, Q4: Q_Photo_NPN, LED_THT:LED_D5.0mm_Clear, symbol Device:Q_Photo_NPN
- added R10, R7, R8, R9: 10k ohm, symbol Device:R
- added R2, R3, R4: 120 ohm, symbol Device:R
- added R5: 100 ohm, symbol Device:R
- added R6: 100k ohm, symbol Device:R
- J6: footprint Connector_PinHeader_2.54mm:PinHeader_1x02_P2.54mm_Vertical -> footprints:YAAJ_DCDC_StepDown_LM2596
- R1: value 100 ohm -> 120 ohm
Connections:
- net BUCK +: now also R1.1, R2.1, R3.1, R4.1
- net GND: now also J15.2 (Pin_2), Q1.2 (E), Q2.2 (E), Q3.2 (E), Q4.2 (E), R6.1
- net IR 1: now also Q1.1 (C), R7.2
- net IR 2: now also Q2.1 (C), R8.2
- net IR 3: now also Q3.1 (C), R9.2
- net IR 4: now also Q4.1 (C), R10.2
- net IR EM: now also R5.1; no longer R1.1
- net at R1.2: now also D1.2 (A)
- net 3V3: now reaches J13.1 (Pin_1)
- net 3V3: now also R10.1, R7.1, R8.1, R9.1
- new net: D1.1 (K), D2.1 (K), D3.1 (K), D4.1 (K), J15.3 (Pin_3)
- new net: D4.2 (A), R4.2
- new net: D2.2 (A), R2.2
- new net: J15.1 (Pin_1), R5.2, R6.2
- new net: D3.2 (A), R3.2
- no-connect marks 16 -> 15
Other:
- note added: "IR EMITTERS"
- note added: "IR RECEIVER"
- note removed: "IR SENSORS"
- moved on the sheet: R1
