File: kiCad/schema/schema.kicad_sch (KiCad schematic)
At the start: 31 parts, among them J1 Conn_01x06_Pin, J11 Switch, J12 Conn_01x15_Pin, J13 Conn_01x15_Pin, J14 Conn_01x06_Pin, J15 MOSFET, J3 M1 Right, J4 M2 Left, J5 Bat, J6 Buck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

Commit message: Day 14 -- whole schematics done with footprints
Parts:
- J15: footprint (none) -> footprints:SOT95P280X125-3N
- R1, R10, R2, R3, R4, R5, R6, R7, R8, R9: footprint (none) -> Resistor_THT:R_Axial_DIN0207_L6.3mm_D2.5mm_P7.62mm_Horizontal
Connections:
- net IR EM: now also J12.12 (Pin_12)
- no-connect marks 15 -> 14
Other:
- moved on the sheet: C3
Changed lines of the file:
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@@
 	)
 	(junction
+		(at 185.42 77.47)
+		(diameter 0)
+		(color 0 0 0 0)
+	)
+	(junction
+		(at 185.42 69.85)
+		(diameter 0)
+		(color 0 0 0 0)
+	)
+	(junction
 		(at 92.71 105.41)
 		(diameter 0)
@@
 	)
 	(junction
-		(at 184.15 69.85)
-		(diameter 0)
-		(color 0 0 0 0)
-	)
-	(junction
 		(at 236.22 92.71)
 		(diameter 0)
@@
 	)
 	(junction
-		(at 184.15 77.47)
-		(diameter 0)
-		(color 0 0 0 0)
-	)
-	(junction
 		(at 44.45 151.13)
 		(diameter 0)
@@
 	)
 	(no_connect
-		(at 105.41 93.98)
-	)
-	(no_connect
 		(at 111.76 78.74)
 	)
@@
 	(wire
 		(pts
-			(xy 181.61 69.85) (xy 184.15 69.85)
+			(xy 181.61 69.85) (xy 185.42 69.85)
 		)
 		(stroke
@@
 	(wire
 		(pts
-			(xy 184.15 69.85) (xy 187.96 69.85)
+			(xy 185.42 69.85) (xy 189.23 69.85)
 		)
 		(stroke
@@
 	(wire
 		(pts
-			(xy 184.15 77.47) (xy 187.96 77.47)
+			(xy 185.42 77.47) (xy 189.23 77.47)
 		)
 		(stroke
@@
 	(wire
 		(pts
+			(xy 88.9 93.98) (xy 105.41 93.98)
+		)
+		(stroke
+			(width 0)
+			(type default)
+		)
+	)
+	(wire
+		(pts
 			(xy 156.21 69.85) (xy 167.64 69.85)
 		)
@@
 	(wire
 		(pts
-			(xy 181.61 77.47) (xy 184.15 77.47)
+			(xy 181.61 77.47) (xy 185.42 77.47)
 		)
 		(stroke
@@
 	)
 	(label "GND"
-		(at 187.96 69.85 0)
+		(at 189.23 69.85 0)
 		(effects
 			(font
@@
 	)
 	(label "IR EM"
+		(at 88.9 93.98 0)
+		(effects
+			(font
+				(size 1.27 1.27)
+			)
+			(justify left bottom)
+		)
+	)
+	(label "IR EM"
 		(at 223.52 92.71 180)
 		(effects
@@
 	)
 	(label "BAT +"
-		(at 187.96 77.47 0)
+		(at 189.23 77.47 0)
 		(effects
 			(font
@@
 			)
 		)
-		(property "Footprint" ""
+		(property "Footprint" "Resistor_THT:R_Axial_DIN0207_L6.3mm_D2.5mm_P7.62mm_Horizontal"
 			(at 238.252 67.31 90)
 			(hide yes)
@@
 			)
 		)
-		(property "Footprint" ""
+		(property "Footprint" "Resistor_THT:R_Axial_DIN0207_L6.3mm_D2.5mm_P7.62mm_Horizontal"
 			(at 225.552 67.31 90)
 			(hide yes)
@@
 			)
 		)
-		(property "Footprint" ""
+		(property "Footprint" "footprints:SOT95P280X125-3N"
 			(at 250.19 92.71 0)
 			(hide yes)
@@
 			)
 		)
-		(property "Footprint" ""
+		(property "Footprint" "Resistor_THT:R_Axial_DIN0207_L6.3mm_D2.5mm_P7.62mm_Horizontal"
 			(at 60.452 144.78 90)
 			(hide yes)
@@
 			)
 		)
-		(property "Footprint" ""
+		(property "Footprint" "Resistor_THT:R_Axial_DIN0207_L6.3mm_D2.5mm_P7.62mm_Horizontal"
 			(at 42.672 144.78 90)
 			(hide yes)
@@
 	(symbol
 		(lib_id "Device:C")
-		(at 184.15 73.66 0)
+		(at 185.42 73.66 0)
 		(unit 1)
 		(body_style 1)
@@
 		(dnp no)
 		(property "Reference" "C3"
-			(at 185.166 66.294 0)
+			(at 186.436 66.294 0)
 			(show_name no)
 			(do_not_autoplace no)
@@
 		)
 		(property "Value" "C"
-			(at 185.166 68.834 0)
+			(at 186.436 68.834 0)
 			(show_name no)
 			(do_not_autoplace no)
@@
 		)
 		(property "Footprint" "Capacitor_THT:C_Disc_D3.0mm_W1.6mm_P2.50mm"
-			(at 185.1152 77.47 0)
+			(at 186.3852 77.47 0)
 			(hide yes)
 			(show_name no)
@@
 		)
 		(property "Datasheet" ""
-			(at 184.15 73.66 0)
+			(at 185.42 73.66 0)
 			(hide yes)
 			(show_name no)
@@
 		)
 		(property "Description" "Unpolarized capacitor"
-			(at 184.15 73.66 0)
+			(at 185.42 73.66 0)
 			(hide yes)
 			(show_name no)
@@
 			)
 		)
-		(property "Footprint" ""
+		(property "Footprint" "Resistor_THT:R_Axial_DIN0207_L6.3mm_D2.5mm_P7.62mm_Horizontal"
 			(at 237.998 100.33 90)
 			(hide yes)
@@
 			)
 		)
-		(property "Footprint" ""
+		(property "Footprint" "Resistor_THT:R_Axial_DIN0207_L6.3mm_D2.5mm_P7.62mm_Horizontal"
 			(at 26.162 144.78 90)
 			(hide yes)
@@
 			)
 		)
-		(property "Footprint" ""
+		(property "Footprint" "Resistor_THT:R_Axial_DIN0207_L6.3mm_D2.5mm_P7.62mm_Horizontal"
 			(at 262.382 67.31 90)
 			(hide yes)
@@
 			)
 		)
-		(property "Footprint" ""
+		(property "Footprint" "Resistor_THT:R_Axial_DIN0207_L6.3mm_D2.5mm_P7.62mm_Horizontal"
 			(at 76.962 144.78 90)
 			(hide yes)
@@
 			)
 		)
-		(property "Footprint" ""
+		(property "Footprint" "Resistor_THT:R_Axial_DIN0207_L6.3mm_D2.5mm_P7.62mm_Horizontal"
 			(at 250.952 67.31 90)
 			(hide yes)
@@
 		(dnp no)
 		(property "Reference" "C1"
-			(at 93.726 94.234 0)
+			(at 89.916 96.52 0)
 			(show_name no)
 			(do_not_autoplace no)
@@
 			)
 		)
-		(property "Footprint" ""
+		(property "Footprint" "Resistor_THT:R_Axial_DIN0207_L6.3mm_D2.5mm_P7.62mm_Horizontal"
 			(at 229.87 94.488 90)
 			(hide yes)
