File: kiCad/schema/schema.kicad_sch (KiCad schematic)
At the start: 31 parts, among them J1 Conn_01x06_Pin, J11 Switch, J12 Conn_01x15_Pin, J13 Conn_01x15_Pin, J14 Conn_01x06_Pin, J15 MOSFET, J3 M1 Right, J4 M2 Left, J5 Bat, J6 Buck, Q1 Q_Photo_NPN, Q2 Q_Photo_NPN, Q3 Q_Photo_NPN, Q4 Q_Photo_NPN

Commit message: Day 16 - PCB layout
Parts:
- removed J12, J13: Conn_01x15_Pin, Connector_PinHeader_2.54mm:PinHeader_1x15_P2.54mm_Vertical, symbol Connector:Conn_01x15_Pin
- added J2: Esp32, footprints:MODULE_ESP32_DEVKIT_V1, symbol Connector_Generic:Conn_02x15_Counter_Clockwise
Connections:
- net 3V3: now also J2.30 (Pin_30)
- net AIN 1: now also J2.8 (Pin_8)
- net AIN 2: now also J2.7 (Pin_7)
- net BIN 1: now also J2.6 (Pin_6)
- net BIN 2: now also J2.5 (Pin_5)
- net BUCK +: now also J2.2 (Pin_2)
- net ENC A1: now also J2.12 (Pin_12)
- net ENC A2: now also J2.11 (Pin_11)
- net ENC B1: now also J2.10 (Pin_10)
- net ENC B2: now also J2.9 (Pin_9)
- net GND: now also J2.1 (Pin_1), J2.29 (Pin_29)
- net IR 1: now also J2.14 (Pin_14)
- net IR 2: now also J2.13 (Pin_13)
- net IR 3: now also J2.26 (Pin_26)
- net IR 4: now also J2.23 (Pin_23)
- net IR EM: now also J2.4 (Pin_4)
Other:
- moved on the sheet: C1, C2

Commit message: Day 17 - Started routing
Parts:
- removed J5: Bat, Connector_JST:JST_PH_B2B-PH-K_1x02_P2.00mm_Vertical, symbol Connector_Generic:Conn_01x02
- added J5: Bat, TerminalBlock:TerminalBlock_MaiXu_MX126-5.0-02P_1x02_P5.00mm, symbol Connector:Screw_Terminal_01x02
- J3, J4: footprint Connector_PinHeader_2.54mm:PinHeader_1x06_P2.54mm_Vertical -> Connector_PinSocket_2.54mm:PinSocket_1x06_P2.54mm_Vertical
Connections:
- net 3V3: now also J1.1 (Pin_1)
- net BAT R+: now also J5.1 (Pin_1)
- net BUCK +: no longer J1.1 (Pin_1)
- net GND: now also J5.2 (Pin_2)

Commit message: Day 19 - PCB done
Connections:
- net BUCK +: now also C1.1, C2.2, J2.1 (Pin_1); no longer C1.2, C2.1, J2.2 (Pin_2)
- net GND: now also C1.2, C2.1, J2.2 (Pin_2); no longer C1.1, C2.2, J2.1 (Pin_1)
- net IR 1: now also J2.18 (Pin_18); no longer J2.14 (Pin_14)
- net IR 2: now also J2.27 (Pin_27); no longer J2.13 (Pin_13)
- net IR 3: now also J2.19 (Pin_19); no longer J2.26 (Pin_26)
- net IR 4: now also J2.26 (Pin_26); no longer J2.23 (Pin_23)
- net IR EM: now also J2.28 (Pin_28); no longer J2.4 (Pin_4)
Changed lines of the file:
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@@
-	)
-	(no_connect
-		(at 116.84 97.79)
 	)
 	(no_connect
@@
 	)
 	(no_connect
-		(at 116.84 72.39)
+		(at 104.14 74.93)
 	)
 	(no_connect
@@
 	)
 	(no_connect
-		(at 116.84 74.93)
+		(at 116.84 85.09)
 	)
 	(no_connect
-		(at 116.84 95.25)
+		(at 104.14 97.79)
 	)
 	(no_connect
@@
 	)
 	(no_connect
+		(at 104.14 100.33)
+	)
+	(no_connect
 		(at 167.64 80.01)
 	)
@@
 	(wire
 		(pts
-			(xy 95.25 97.79) (xy 104.14 97.79)
-		)
-		(stroke
-			(width 0)
-			(type default)
-		)
-	)
-	(wire
-		(pts
 			(xy 156.21 77.47) (xy 167.64 77.47)
 		)
@@
 	(wire
 		(pts
-			(xy 97.79 74.93) (xy 104.14 74.93)
-		)
-		(stroke
-			(width 0)
-			(type default)
-		)
-	)
-	(wire
-		(pts
 			(xy 240.03 63.5) (xy 252.73 63.5)
 		)
@@
 	(wire
 		(pts
+			(xy 116.84 74.93) (xy 121.92 74.93)
+		)
+		(stroke
+			(width 0)
+			(type default)
+		)
+	)
+	(wire
+		(pts
 			(xy 223.52 92.71) (xy 226.06 92.71)
 		)
@@
 	(wire
 		(pts
+			(xy 116.84 77.47) (xy 121.92 77.47)
+		)
+		(stroke
+			(width 0)
+			(type default)
+		)
+	)
+	(wire
+		(pts
 			(xy 97.79 77.47) (xy 104.14 77.47)
 		)
@@
 	(wire
 		(pts
-			(xy 116.84 85.09) (xy 121.92 85.09)
-		)
-		(stroke
-			(width 0)
-			(type default)
-		)
-	)
-	(wire
-		(pts
 			(xy 49.53 93.98) (xy 58.42 93.98)
 		)
@@
 	(wire
 		(pts
+			(xy 116.84 95.25) (xy 121.92 95.25)
+		)
+		(stroke
+			(width 0)
+			(type default)
+		)
+	)
+	(wire
+		(pts
 			(xy 181.61 77.47) (xy 185.42 77.47)
 		)
@@
 	(wire
 		(pts
-			(xy 95.25 100.33) (xy 104.14 100.33)
-		)
-		(stroke
-			(width 0)
-			(type default)
-		)
-	)
-	(wire
-		(pts
 			(xy 171.45 72.39) (xy 181.61 72.39)
 		)
@@
 	(wire
 		(pts
+			(xy 116.84 97.79) (xy 121.92 97.79)
+		)
+		(stroke
+			(width 0)
+			(type default)
+		)
+	)
+	(wire
+		(pts
 			(xy 86.36 73.66) (xy 92.71 73.66)
 		)
@@
 	(wire
 		(pts
+			(xy 116.84 72.39) (xy 121.92 72.39)
+		)
+		(stroke
+			(width 0)
+			(type default)
+		)
+	)
+	(wire
+		(pts
 			(xy 62.23 151.13) (xy 62.23 153.67)
-		)
-		(stroke
-			(width 0)
-			(type default)
-		)
-	)
-	(wire
-		(pts
-			(xy 116.84 77.47) (xy 121.92 77.47)
 		)
 		(stroke
@@
 	)
 	(label "IR 4"
-		(at 121.92 85.09 0)
+		(at 121.92 77.47 0)
+		(effects
+			(font
+				(size 1.27 1.27)
+			)
+			(justify left bottom)
+		)
+	)
+	(label "IR 1"
+		(at 121.92 97.79 0)
 		(effects
 			(font
@@
 	)
 	(label "IR EM"
-		(at 97.79 74.93 0)
+		(at 121.92 72.39 0)
 		(effects
 			(font
@@
 		)
 	)
-	(label "BUCK +"
-		(at 83.82 81.28 0)
-		(effects
-			(font
-				(size 1.27 1.27)
-			)
-			(justify left bottom)
-		)
-	)
 	(label "AOUT 2"
 		(at 156.21 72.39 180)
@@
 		)
 	)
+	(label "GND"
+		(at 83.82 81.28 0)
+		(effects
+			(font
+				(size 1.27 1.27)
+			)
+			(justify left bottom)
+		)
+	)
 	(label "3V3"
 		(at 44.45 135.89 0)
@@
 		)
 	)
-	(label "GND"
-		(at 82.55 64.77 0)
+	(label "IR 2"
+		(at 121.92 74.93 0)
 		(effects
 			(font
@@
 		)
 	)
-	(label "IR 1"
-		(at 95.25 100.33 0)
-		(effects
-			(font
-				(size 1.27 1.27)
-			)
-			(justify left bottom)
-		)
-	)
 	(label "AIN 1"
 		(at 97.79 85.09 0)
@@
 		)
 	)
-	(label "IR 2"
-		(at 95.25 97.79 0)
-		(effects
-			(font
-				(size 1.27 1.27)
-			)
-			(justify left bottom)
-		)
-	)
 	(label "BOUT 1"
 		(at 160.02 90.17 0)
@@
 		)
 	)
+	(label "BUCK +"
+		(at 82.55 64.77 0)
+		(effects
+			(font
+				(size 1.27 1.27)
+			)
+			(justify left bottom)
+		)
+	)
 	(label "ENC B2"
 		(at 95.25 87.63 0)
@@
 	)
 	(label "IR 3"
-		(at 121.92 77.47 0)
-		(effects
-			(font
+		(at 121.92 95.25 0)
+		(effects
+			(font

Commit message: Day 20 - Solved esp32 mis-pin alignment
Parts:
- added R11: 10k ohm, Resistor_THT:R_Axial_DIN0207_L6.3mm_D2.5mm_P7.62mm_Horizontal, symbol Device:R
Connections:
- net 3V3: now also J2.15 (Pin_15); no longer J2.30 (Pin_30)
- net AIN 1: now also J2.23 (Pin_23); no longer J2.8 (Pin_8)
- net AIN 2: now also J2.22 (Pin_22); no longer J2.7 (Pin_7)
- net BIN 1: now also J2.21 (Pin_21); no longer J2.6 (Pin_6)
- net BIN 2: now also J2.20 (Pin_20); no longer J2.5 (Pin_5)
- net BUCK +: now also J2.16 (Pin_16); no longer J2.1 (Pin_1)
- net ENC A1: now also J2.27 (Pin_27); no longer J2.12 (Pin_12)
- net ENC A2: now also J2.26 (Pin_26); no longer J2.11 (Pin_11)
- net ENC B1: now also J2.25 (Pin_25); no longer J2.10 (Pin_10)
- net ENC B2: now also J2.24 (Pin_24); no longer J2.9 (Pin_9)
- net GND: now also J2.14 (Pin_14), J2.17 (Pin_17); no longer J2.2 (Pin_2), J2.29 (Pin_29)
- net IR 1: now also J2.3 (Pin_3); no longer J2.18 (Pin_18)
- net IR 2: now also J2.12 (Pin_12); no longer J2.27 (Pin_27)
- net IR 3: now also J2.4 (Pin_4); no longer J2.19 (Pin_19)
- net IR 4: now also J2.11 (Pin_11); no longer J2.26 (Pin_26)
- net IR EM: now also J2.13 (Pin_13); no longer J2.28 (Pin_28)
Other:
- moved on the sheet: J2

Commit message: Day 21 - esp32 misalignment fixed
Connections:
- net 3V3: now also J2.1 (Pin_1); no longer J2.15 (Pin_15)
- net AIN 2: now also J2.24 (Pin_24); no longer J2.22 (Pin_22)
- net BIN 1: now also J2.25 (Pin_25); no longer J2.21 (Pin_21)
- net BIN 2: now also J2.26 (Pin_26); no longer J2.20 (Pin_20)
- net BUCK +: now also J2.30 (Pin_30); no longer J2.16 (Pin_16)
- net ENC A1: now also J2.19 (Pin_19); no longer J2.27 (Pin_27)
- net ENC A2: now also J2.20 (Pin_20); no longer J2.26 (Pin_26)
- net ENC B1: now also J2.21 (Pin_21); no longer J2.25 (Pin_25)
- net ENC B2: now also J2.22 (Pin_22); no longer J2.24 (Pin_24)
- net GND: now also J2.2 (Pin_2), J2.29 (Pin_29); no longer J2.14 (Pin_14), J2.17 (Pin_17)
- net IR 1: now also J2.13 (Pin_13); no longer J2.3 (Pin_3)
- net IR 2: now also J2.4 (Pin_4); no longer J2.12 (Pin_12)
- net IR 3: now also J2.12 (Pin_12); no longer J2.4 (Pin_4)
- net IR 4: now also J2.5 (Pin_5); no longer J2.11 (Pin_11)
- net IR EM: now also J2.3 (Pin_3); no longer J2.13 (Pin_13)
Other:
- moved on the sheet: J2

Commit message: Day 23: Added tactile button, boost conv
Parts:
- removed R11: 10k ohm, Resistor_THT:R_Axial_DIN0207_L6.3mm_D2.5mm_P7.62mm_Horizontal, symbol Device:R
- added J7: Tact Switch, Button_Switch_THT:SW_PUSH_6mm_H5mm, symbol Connector:Conn_01x02_Pin
- C1, C3: value C -> C 0.1
- C2: value C_Polarized -> C_Polarized 47; footprint Capacitor_THT:CP_Radial_D4.0mm_P1.50mm -> Capacitor_THT:CP_Radial_D6.3mm_P2.50mm
- J6: value Buck -> BOOST; footprint footprints:YAAJ_DCDC_StepDown_LM2596 -> footprints:TPS61023
Connections:
- net GND: now also J6.3 (Pin_3), J7.2 (Pin_2); no longer J6.4 (Pin_4)
- net SW PIN: now reaches J2.28 (Pin_28)
- net SW PIN: now also J7.1 (Pin_1)
- net BUCK + renamed BOOST +
- net BOOST +: now also J6.4 (Pin_4); no longer J6.3 (Pin_3)
- no-connect marks 14 -> 13
Other:
- moved on the sheet: J6

Commit message: Day 24 -- Final commit on V1
Parts:
- R1, R2, R3, R4: value 120 ohm -> 220 ohm
Connections:
- net BAT +: now also C3.1, J14.4 (Pin_4); no longer C3.2, J14.3 (Pin_3)
- net GND: now also C3.2, J14.3 (Pin_3); no longer C3.1, J14.4 (Pin_4)
Changed lines of the file:
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@@
 	)
 	(junction
-		(at 185.42 69.85)
+		(at 92.71 73.66)
 		(diameter 0)
 		(color 0 0 0 0)
 	)
 	(junction
-		(at 92.71 73.66)
+		(at 185.42 69.85)
 		(diameter 0)
 		(color 0 0 0 0)
@@
 	(wire
 		(pts
+			(xy 189.23 69.85) (xy 185.42 69.85)
+		)
+		(stroke
+			(width 0)
+			(type default)
+		)
+	)
+	(wire
+		(pts
 			(xy 83.82 73.66) (xy 86.36 73.66)
 		)
@@
 	(wire
 		(pts
-			(xy 185.42 69.85) (xy 189.23 69.85)
-		)
-		(stroke
-			(width 0)
-			(type default)
-		)
-	)
-	(wire
-		(pts
 			(xy 181.61 72.39) (xy 181.61 69.85)
 		)
@@
 	(wire
 		(pts
-			(xy 185.42 77.47) (xy 189.23 77.47)
-		)
-		(stroke
-			(width 0)
-			(type default)
-		)
-	)
-	(wire
-		(pts
 			(xy 185.42 102.87) (xy 190.5 102.87)
 		)
@@
 	(wire
 		(pts
+			(xy 189.23 77.47) (xy 185.42 77.47)
+		)
+		(stroke
+			(width 0)
+			(type default)
+		)
+	)
+	(wire
+		(pts
 			(xy 181.61 74.93) (xy 181.61 77.47)
 		)
@@
 	)
 	(label "GND"
-		(at 189.23 69.85 0)
+		(at 189.23 77.47 0)
 		(effects
 			(font
@@
 	)
 	(label "BAT +"
-		(at 189.23 77.47 0)
+		(at 189.23 69.85 0)
 		(effects
 			(font
@@
 			)
 		)
-		(property "Value" "120 ohm"
+		(property "Value" "220 ohm"
 			(at 241.808 68.326 0)
 			(show_name no)
@@
 			)
 		)
-		(property "Value" "120 ohm"
+		(property "Value" "220 ohm"
 			(at 229.108 68.326 0)
 			(show_name no)
@@
 			)
 		)
-		(property "Value" "120 ohm"
+		(property "Value" "220 ohm"
 			(at 265.43 68.072 0)
 			(show_name no)
@@
 			)
 		)
-		(property "Value" "120 ohm"
+		(property "Value" "220 ohm"
 			(at 254 68.072 0)
 			(show_name no)
