File: kiCad/schema/schema.kicad_pcb (KiCad board)
At the start: 2 copper layers, 1 part, among them J1 Esp32

Commit message: Day 10 - CAD design, PCB design started
Parts:
- removed J1: Esp32, Connector_PinHeader_2.54mm:PinHeader_1x15_P2.54mm_Vertical
- added J12: Conn_01x15_Pin, Connector_PinHeader_2.54mm:PinHeader_1x15_P2.54mm_Vertical, F.Cu at (149.8, 86.6)
- added J13: Conn_01x15_Pin, Connector_PinHeader_2.54mm:PinHeader_1x15_P2.54mm_Vertical, F.Cu at (175.3, 122.2)

Commit message: Day 11 -- PCB, footprints, headache
Parts:
- added C1: C, Capacitor_THT:C_Disc_D3.0mm_W1.6mm_P2.50mm, F.Cu at (102.9, 157.9)
- added C2: C_Polarized, Capacitor_THT:CP_Radial_D4.0mm_P1.50mm, F.Cu at (103.4, 165.4)
- added C3: C, Capacitor_THT:C_Disc_D3.0mm_W1.6mm_P2.50mm, F.Cu at (102.9, 161.0)
- added J3: M1 Right, Connector_PinHeader_2.54mm:PinHeader_1x06_P2.54mm_Vertical, F.Cu at (32.8, 141.5)
- added J4: M2 Left, Connector_PinHeader_2.54mm:PinHeader_1x06_P2.54mm_Vertical, F.Cu at (116.3, 139.2)
- moved J13 121.5 mm to (58.7, 156.4), turned to 90 degrees
- moved J12 117.7 mm to (58.7, 161.0), turned to 90 degrees
Other:
- board outline added: 103.8 x 139.4 mm

Commit message: Day 12 -- Resuming the project
Parts:
- added J1: Conn_01x06_Pin, Connector_PinHeader_2.54mm:PinHeader_1x06_P2.54mm_Vertical, F.Cu at (71.9, 110.8)
- added J11: Switch, Button_Switch_THT:SW_Slide_SPDT_Straight_CK_OS102011MS2Q, F.Cu at (64.4, 75.9)
- added J14: Conn_01x06_Pin, Connector_PinHeader_2.54mm:PinHeader_1x06_P2.54mm_Vertical, F.Cu at (76.5, 110.8)
- added J5: Bat, Connector_JST:JST_PH_B2B-PH-K_1x02_P2.00mm_Vertical, F.Cu at (53.3, 63.7)
- added J6: Buck, Connector_PinHeader_2.54mm:PinHeader_1x02_P2.54mm_Vertical, F.Cu at (92.2, 99.1)

Commit message: Day 13 -- IR leds, footprints
Parts:
- added D1: LED, LED_THT:LED_D5.0mm_Clear, F.Cu at (40.6, 51.8)
- added D2: LED, LED_THT:LED_D5.0mm_Clear, F.Cu at (59.7, 40.4)
- added D3: LED, LED_THT:LED_D5.0mm_Clear, F.Cu at (81.5, 39.6)
- added D4: LED, LED_THT:LED_D5.0mm_Clear, F.Cu at (104.1, 50.8)
- added Q1: Q_Photo_NPN, LED_THT:LED_D5.0mm_Clear, F.Cu at (48.0, 49.0)
- added Q2: Q_Photo_NPN, LED_THT:LED_D5.0mm_Clear, F.Cu at (67.1, 40.6)
- added Q3: Q_Photo_NPN, LED_THT:LED_D5.0mm_Clear, F.Cu at (88.9, 40.9)
- added Q4: Q_Photo_NPN, LED_THT:LED_D5.0mm_Clear, F.Cu at (111.5, 56.9)
- J6: footprint Connector_PinHeader_2.54mm:PinHeader_1x02_P2.54mm_Vertical -> footprints:YAAJ_DCDC_StepDown_LM2596
- moved J6 22.9 mm to (77.2, 81.8)
- moved J5 8.49 mm to (45.7, 67.6)
Connections:
- J13 pad 1: unconnected-(J13-Pin_1-Pad1) -> /3V3

Commit message: Day 14 -- whole schematics done with footprints
Parts:
- added J15: MOSFET, footprints:SOT95P280X125-3N, F.Cu at (118.4, 88.8)
- added R1: 120 ohm, Resistor_THT:R_Axial_DIN0207_L6.3mm_D2.5mm_P7.62mm_Horizontal, F.Cu at (73.0, 67.0)
- added R10: 10k ohm, Resistor_THT:R_Axial_DIN0207_L6.3mm_D2.5mm_P7.62mm_Horizontal, F.Cu at (73.0, 103.5)
- added R2: 120 ohm, Resistor_THT:R_Axial_DIN0207_L6.3mm_D2.5mm_P7.62mm_Horizontal, F.Cu at (73.0, 71.1)
- added R3: 120 ohm, Resistor_THT:R_Axial_DIN0207_L6.3mm_D2.5mm_P7.62mm_Horizontal, F.Cu at (73.0, 75.1)
- added R4: 120 ohm, Resistor_THT:R_Axial_DIN0207_L6.3mm_D2.5mm_P7.62mm_Horizontal, F.Cu at (73.0, 79.2)
- added R5: 100 ohm, Resistor_THT:R_Axial_DIN0207_L6.3mm_D2.5mm_P7.62mm_Horizontal, F.Cu at (73.0, 83.2)
- added R6: 100k ohm, Resistor_THT:R_Axial_DIN0207_L6.3mm_D2.5mm_P7.62mm_Horizontal, F.Cu at (73.0, 87.3)
- added R7: 10k ohm, Resistor_THT:R_Axial_DIN0207_L6.3mm_D2.5mm_P7.62mm_Horizontal, F.Cu at (73.0, 91.3)
- added R8: 10k ohm, Resistor_THT:R_Axial_DIN0207_L6.3mm_D2.5mm_P7.62mm_Horizontal, F.Cu at (73.0, 95.4)
- added R9: 10k ohm, Resistor_THT:R_Axial_DIN0207_L6.3mm_D2.5mm_P7.62mm_Horizontal, F.Cu at (73.0, 99.4)
- moved J12 97.2 mm to (84.4, 67.3), turned to 0 degrees
- moved J13 94.2 mm to (89.0, 67.3), turned to 0 degrees
- moved J3 88.3 mm to (98.2, 82.2)
- moved C1 70.3 mm to (111.3, 88.1)
- moved C2 70.3 mm to (111.8, 95.6)
- moved C3 70.3 mm to (111.3, 91.2)
- moved J5 68.6 mm to (112.7, 82.7)
- moved Q1 63.9 mm to (108.8, 68.7)
- moved J4 58.5 mm to (102.8, 82.2)
- moved D1 55.8 mm to (93.8, 68.7)
- moved Q2 54.8 mm to (108.8, 76.2)
- moved D2 49.5 mm to (93.8, 76.2)
- moved J14 42.1 mm to (107.4, 82.2)
- moved J11 39.6 mm to (95.3, 100.8)
- moved Q3 39.0 mm to (116.2, 68.7)
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Connections:
- J12 pad 12: unconnected-(J12-Pin_12-Pad12) -> /IR EM
Other:
- board outline removed

Commit message: Day 14 -- PCB layout
Parts:
- moved J6 83.1 mm to (81.0, 127.3)
- moved R10 69.2 mm to (135.6, 74.2), turned to 90 degrees
- moved R9 65.8 mm to (121.2, 54.6), turned to 90 degrees
- moved R4 57.3 mm to (130.0, 74.4), turned to 90 degrees
- moved R6 55.6 mm to (128.5, 87.4)
- moved J5 47.9 mm to (65.3, 75.9)
- moved R3 47.6 mm to (116.1, 54.9), turned to 90 degrees
- moved J11 47.1 mm to (137.0, 78.7)
- moved R8 44.1 mm to (94.0, 56.6), turned to 90 degrees
- moved R5 41.2 mm to (114.0, 86.1)
- moved Q2 41.1 mm to (92.2, 38.6)
- moved Q1 39.3 mm to (72.9, 52.6), turned to 45 degrees
- moved D2 39.0 mm to (82.5, 38.9)
- moved D4 37.6 mm to (131.0, 53.3), turned to -45 degrees
- moved D3 32.3 mm to (112.8, 38.6)
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Other:
- board outline added: 90 x 127.1 mm
