File: kiCad/schema/schema.kicad_pcb (KiCad board)
At the start: 2 copper layers, 90 x 127.1 mm, 31 parts, among them J1 Conn_01x06_Pin, J11 Switch, J12 Conn_01x15_Pin, J13 Conn_01x15_Pin, J14 Conn_01x06_Pin, J15 MOSFET, J3 M1 Right, J4 M2 Left, J5 Bat, J6 Buck, Q1 Q_Photo_NPN, Q2 Q_Photo_NPN, Q3 Q_Photo_NPN, Q4 Q_Photo_NPN

Commit message: Day 16 - PCB layout
Parts:
- removed J12, J13: Conn_01x15_Pin, Connector_PinHeader_2.54mm:PinHeader_1x15_P2.54mm_Vertical
- added J2: Esp32, footprints:MODULE_ESP32_DEVKIT_V1, F.Cu at (101.9, 90.4)
- moved J11 89.4 mm to (67.1, 134.6)
- moved J5 67.1 mm to (67.3, 143.0)
- moved J1 41.3 mm to (93.2, 109.2)
- moved J14 41.2 mm to (111.3, 109.2)
- moved C3 40.9 mm to (114.8, 116.6)
- moved C2 38.4 mm to (115.3, 69.3), turned to 0 degrees
- moved R5 34.7 mm to (86.1, 65.5)
- moved J15 34.7 mm to (97.8, 60.2)
- moved R6 34.7 mm to (100.6, 66.8)
- moved C1 30.6 mm to (117.4, 73.7), turned to 180 degrees
- moved J3 5.93 mm to (84.8, 110.7)
- moved J4 5.45 mm to (119.9, 110.7)
- moved J6 3.34 mm to (80.5, 130.6)

Commit message: Day 17 - Started routing
Parts:
- J3, J4: footprint Connector_PinHeader_2.54mm:PinHeader_1x06_P2.54mm_Vertical -> Connector_PinSocket_2.54mm:PinSocket_1x06_P2.54mm_Vertical
- J5: footprint Connector_JST:JST_PH_B2B-PH-K_1x02_P2.00mm_Vertical -> TerminalBlock:TerminalBlock_MaiXu_MX126-5.0-02P_1x02_P5.00mm
- moved R5 14.2 mm to (100.1, 67.8)
- moved J15 8.33 mm to (102.9, 53.6)
- moved R6 5.86 mm to (100.1, 61.0)
- moved J5 1.83 mm to (67.1, 144.8)
- turned J2 to 90 degrees
Connections:
- J1 pad 1: /BUCK + -> /3V3
Routing:
- net /BUCK +: track 0.00 -> 71.8 mm
- net /BOUT 1: track 0.00 -> 33.2 mm
- net /BOUT 2: track 0.00 -> 30.0 mm
- net /AOUT 2: track 0.00 -> 15.2 mm
- net /BAT +: track 0.00 -> 13.1 mm
- net /BAT R+: track 0.00 -> 10.2 mm
- net /GND: track 0.00 -> 9.85 mm
- net /AOUT 1: track 0.00 -> 8.80 mm
