File: kiCad/schema/schema.kicad_pcb (KiCad board)
At the start: 2 copper layers, 90 x 127.1 mm, 33 parts, among them J1 DRV8833, J14 GND, J15 MOSFET, Q1 Q_Photo_NPN, Q2 Q_Photo_NPN, Q3 Q_Photo_NPN, Q4 Q_Photo_NPN

Commit message: Add: CAD design, motor mount, PCB corrections
Parts:
- added Motor mount: MountingHole_3.2mm_M3, MountingHole:MountingHole_3.2mm_M3, F.Cu at (135.2, 131.6)
- added Motor mount - ball: MountingHole_2.5mm, MountingHole:MountingHole_2.5mm, F.Cu at (94.6, 45.2)
- added Motor mount - ball: MountingHole_2.5mm, MountingHole:MountingHole_2.5mm, F.Cu at (114.2, 45.2)
- added Motor mount: MountingHole_3.2mm_M3, MountingHole:MountingHole_3.2mm_M3, F.Cu at (69.4, 114.0)
- moved Switch 14.6 mm to (80.0, 141.6), turned to -90 degrees
- moved Motor mount 12.0 mm to (69.4, 131.6)
- moved Motor mount 8.84 mm to (135.2, 114.0)
- moved C1 1.28 mm to (133.0, 105.3)
Routing:
- net /BAT +: track 68.7 -> 55.2 mm
- net /BOOST +: track 401.2 -> 406.8 mm
- net /BAT R+: track 10.2 -> 14.2 mm
